File: nano8825withstep/nano8825withstep.sch (KiCad schematic (older format))
At the start: 14 parts, among them J1 Conn_01x02, J2 Conn_01x04, J3 Conn_01x04, J4 Conn_01x04, SW1 SW_DIP_x03, SW2 SW_DIP_x03, SW3 SW_DIP_x03

Commit message: Added limit and probe connectors
Parts:
- added C4, C5, C6: 100n, Capacitor_THT:C_Disc_D3.0mm_W1.6mm_P2.50mm, symbol Device:C
- added J5, J6, J7: Conn_01x02, Connector_PinSocket_2.54mm:PinSocket_1x02_P2.54mm_Vertical, symbol Connector_Generic:Conn_01x02
- added J8: Conn_01x02_Female, Connector_PinSocket_2.54mm:PinSocket_1x02_P2.54mm_Vertical, symbol Connector_Generic:Conn_01x02_Female
- added R1, R2, R3: 4k7, Resistor_THT:R_Axial_DIN0204_L3.6mm_D1.6mm_P5.08mm_Horizontal, symbol Device:R
- J2, J3, J4: footprint TerminalBlock:TerminalBlock_bornier-4_P5.08mm -> TerminalBlock_Phoenix:TerminalBlock_Phoenix_MPT-0,5-4-2.54_1x04_P2.54mm_Horizontal
Connections:
- wire segments 129 -> 194
