File: nano8825/nano8825.sch (KiCad schematic (older format))
At the start: 24 parts, among them J1 Conn_01x02, J2 Conn_01x04, J3 Conn_01x04, J4 Conn_01x04, J5 Conn_01x02, J6 Conn_01x02, J7 Conn_01x02, J8 Conn_01x02_Female, SW1 SW_DIP_x03, SW2 SW_DIP_x03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

Commit message: Added Output for nano8825 board
Parts:
- J8: symbol Connector_Generic:Conn_01x02_Female -> nano8825-rescue:Conn_01x02_Female-Connector_Generic
Changed lines of the file:
@@
 EESchema Schematic File Version 4
+LIBS:nano8825-cache
 EELAYER 26 0
 EELAYER END
@@
 	4100 5900 4100 6500
 $Comp
-L Connector_Generic:Conn_01x02_Female J8
+L nano8825-rescue:Conn_01x02_Female-Connector_Generic J8
 U 1 1 5AD2DFC9
 P 2000 4450

Commit message: Updated some footprints
Parts:
- SW1, SW2, SW3: footprint Package_DIP:DIP-6_W7.62mm -> Button_Switch_THT:SW_DIP_SPSTx03_Slide_6.7x9.18mm_W7.62mm_P2.54mm_LowProfile
Changed lines of the file:
@@
 F 0 "SW1" H 4500 2600 50  0000 C CNN
 F 1 "SW_DIP_x03" H 4500 2700 50  0000 C CNN
-F 2 "Package_DIP:DIP-6_W7.62mm" H 4500 2900 50  0001 C CNN
+F 2 "Button_Switch_THT:SW_DIP_SPSTx03_Slide_6.7x9.18mm_W7.62mm_P2.54mm_LowProfile" H 4500 2900 50  0001 C CNN
 F 3 "" H 4500 2900 50  0001 C CNN
 	1    4500 2900
@@
 F 0 "SW2" H 4500 4500 50  0000 C CNN
 F 1 "SW_DIP_x03" H 4500 4600 50  0000 C CNN
-F 2 "Package_DIP:DIP-6_W7.62mm" H 4500 4800 50  0001 C CNN
+F 2 "Button_Switch_THT:SW_DIP_SPSTx03_Slide_6.7x9.18mm_W7.62mm_P2.54mm_LowProfile" H 4500 4800 50  0001 C CNN
 F 3 "" H 4500 4800 50  0001 C CNN
 	1    4500 4800
@@
 F 0 "SW3" H 4500 6450 50  0000 C CNN
 F 1 "SW_DIP_x03" H 4500 6550 50  0000 C CNN
-F 2 "Package_DIP:DIP-6_W7.62mm" H 4500 6700 50  0001 C CNN
+F 2 "Button_Switch_THT:SW_DIP_SPSTx03_Slide_6.7x9.18mm_W7.62mm_P2.54mm_LowProfile" H 4500 6700 50  0001 C CNN
 F 3 "" H 4500 6700 50  0001 C CNN
 	1    4500 6700

Commit message: Added Caliper and updated drv8825 board
Other:
- note added: "Probe"
- note added: "X\nLIMIT"
- note added: "Y\nLIMIT"
- note added: "Z LIMIT"
Changed lines of the file:
@@
-$EndComp
-$Comp
-L Switch:SW_DIP_x03 SW1
-U 1 1 5AC2870A
-P 4500 2900
-F 0 "SW1" H 4500 2600 50  0000 C CNN
-F 1 "SW_DIP_x03" H 4500 2700 50  0000 C CNN
-F 2 "Button_Switch_THT:SW_DIP_SPSTx03_Slide_6.7x9.18mm_W7.62mm_P2.54mm_LowProfile" H 4500 2900 50  0001 C CNN
-F 3 "" H 4500 2900 50  0001 C CNN
-	1    4500 2900
-	1    0    0    -1
 $EndComp
 $Comp
@@
 Wire Wire Line
 	4100 4600 4100 4700
-Wire Wire Line
-	4100 2700 4200 2700
 Connection ~ 4100 2700
 Wire Wire Line
 	4100 2700 4100 2800
-Wire Wire Line
-	4100 2800 4200 2800
 Connection ~ 4100 2800
 Wire Wire Line
 	4100 2800 4100 2900
-Wire Wire Line
-	4100 2900 4200 2900
 Connection ~ 4100 2900
 Wire Wire Line
 	4100 2900 4100 3900
-Wire Wire Line
-	4800 2700 5000 2700
-Wire Wire Line
-	4800 2800 5000 2800
-Wire Wire Line
-	4800 2900 5000 2900
 Wire Wire Line
 	4800 4600 5000 4600
@@
 Wire Wire Line
 	1900 4000 1900 4250
+Wire Wire Line
+	4100 2700 4200 2700
+Wire Wire Line
+	4100 2800 4200 2800
+Wire Wire Line
+	4100 2900 4200 2900
+Wire Wire Line
+	4800 2900 5000 2900
+Wire Wire Line
+	4800 2800 5000 2800
+Wire Wire Line
+	4800 2700 5000 2700
+$Comp
+L Switch:SW_DIP_x03 SW1
+U 1 1 5AC2870A
+P 4500 2900
+F 0 "SW1" H 4500 2600 50  0000 C CNN
+F 1 "SW_DIP_x03" H 4500 2700 50  0000 C CNN
+F 2 "Button_Switch_THT:SW_DIP_SPSTx03_Slide_6.7x9.18mm_W7.62mm_P2.54mm_LowProfile" H 4500 2900 50  0001 C CNN
+F 3 "" H 4500 2900 50  0001 C CNN
+	1    4500 2900
+	1    0    0    -1
+$EndComp
+Text Notes 2900 6700 0    50   ~ 0
+Z LIMIT
+Text Notes 2650 6750 0    50   ~ 0
+Y\nLIMIT
+Text Notes 2300 6750 0    50   ~ 0
+X\nLIMIT
+Text Notes 1850 4600 0    50   ~ 0
+Probe
 $EndSCHEMATC

Commit message: Added FAULT line to force fast decay
Connections:
- wire segments 194 -> 200
Changed lines of the file:
@@
 Connection ~ 4100 4800
 Wire Wire Line
-	4100 4800 4100 5800
+	4100 4800 4100 5700
 Wire Wire Line
 	4100 4700 4200 4700
@@
 Connection ~ 4100 2900
 Wire Wire Line
-	4100 2900 4100 3900
+	4100 2900 4100 3800
 Wire Wire Line
 	4800 4600 5000 4600
@@
 Text Notes 1850 4600 0    50   ~ 0
 Probe
+Wire Wire Line
+	5000 3800 4100 3800
+Connection ~ 4100 3800
+Wire Wire Line
+	4100 3800 4100 3900
+Wire Wire Line
+	5000 1900 4100 1900
+Wire Wire Line
+	4100 1900 4100 2000
+Connection ~ 4100 2000
+Wire Wire Line
+	5000 5700 4100 5700
+Connection ~ 4100 5700
+Wire Wire Line
+	4100 5700 4100 5800
 $EndSCHEMATC
