File: digital_caliper/digital_caliper.sch (KiCad schematic (older format))
At the start: 13 parts, among them J1 Conn_01x05, J2 Conn_01x04_Male, Q1 2N3904, Q2 2N7000, Q3 2N7000, Q4 2N3904, Q5 2N3904

Commit message: Added FAULT line to force fast decay
Parts:
- removed J1: Conn_01x05, Connector_PinHeader_2.54mm:PinHeader_1x05_P2.54mm_Horizontal, symbol Connector_Generic:Conn_01x05
- added J1: Conn_01x06, Connector_PinHeader_2.54mm:PinHeader_1x06_P2.54mm_Horizontal, symbol Connector_Generic:Conn_01x06
- C1: footprint Capacitor_THT:C_Disc_D3.0mm_W1.6mm_P2.50mm -> Capacitor_SMD:C_0805_2012Metric
- Q1, Q2, Q3, Q4, Q5: footprint Package_TO_SOT_THT:TO-92_Inline -> Package_TO_SOT_SMD:SOT-23
- R1, R2, R3, R4, R5: footprint Resistor_THT:R_Axial_DIN0204_L3.6mm_D1.6mm_P5.08mm_Horizontal -> Resistor_SMD:R_0805_2012Metric
Connections:
- wire segments 64 -> 66
Changed lines of the file:
@@
 L Transistor_FET:2N7000 Q2
 U 1 1 5B360AD9
-P 6000 2450
-F 0 "Q2" H 6205 2496 50  0000 L CNN
-F 1 "2N7000" H 6205 2405 50  0000 L CNN
-F 2 "Package_TO_SOT_THT:TO-92_Inline" H 6200 2375 50  0001 L CIN
-F 3 "https://www.fairchildsemi.com/datasheets/2N/2N7000.pdf" H 6000 2450 50  0001 L CNN
-	1    6000 2450
+P 5600 2450
+F 0 "Q2" H 5805 2496 50  0000 L CNN
+F 1 "2N7000" H 5805 2405 50  0000 L CNN
+F 2 "Package_TO_SOT_SMD:SOT-23" H 5800 2375 50  0001 L CIN
+F 3 "https://www.fairchildsemi.com/datasheets/2N/2N7000.pdf" H 5600 2450 50  0001 L CNN
+	1    5600 2450
 	1    0    0    -1
 $EndComp
@@
 L Transistor_FET:2N7000 Q3
 U 1 1 5B360B26
-P 6000 3400
-F 0 "Q3" H 6205 3446 50  0000 L CNN
-F 1 "2N7000" H 6205 3355 50  0000 L CNN
-F 2 "Package_TO_SOT_THT:TO-92_Inline" H 6200 3325 50  0001 L CIN
-F 3 "https://www.fairchildsemi.com/datasheets/2N/2N7000.pdf" H 6000 3400 50  0001 L CNN
-	1    6000 3400
+P 5650 3400
+F 0 "Q3" H 5855 3446 50  0000 L CNN
+F 1 "2N7000" H 5855 3355 50  0000 L CNN
+F 2 "Package_TO_SOT_SMD:SOT-23" H 5850 3325 50  0001 L CIN
+F 3 "https://www.fairchildsemi.com/datasheets/2N/2N7000.pdf" H 5650 3400 50  0001 L CNN
+	1    5650 3400
 	1    0    0    -1
 $EndComp
@@
 L Device:R R5
 U 1 1 5B360BC1
-P 5850 3750
-F 0 "R5" V 5643 3750 50  0000 C CNN
-F 1 "100k" V 5734 3750 50  0000 C CNN
-F 2 "Resistor_THT:R_Axial_DIN0204_L3.6mm_D1.6mm_P5.08mm_Horizontal" V 5780 3750 50  0001 C CNN
-F 3 "~" H 5850 3750 50  0001 C CNN
-	1    5850 3750
+P 5950 3750
+F 0 "R5" V 5743 3750 50  0000 C CNN
+F 1 "100k" V 5834 3750 50  0000 C CNN
+F 2 "Resistor_SMD:R_0805_2012Metric" V 5880 3750 50  0001 C CNN
+F 3 "~" H 5950 3750 50  0001 C CNN
+	1    5950 3750
 	0    1    1    0
 $EndComp
@@
 L Device:R R4
 U 1 1 5B360C16
-P 5850 2800
-F 0 "R4" V 5643 2800 50  0000 C CNN
-F 1 "100k" V 5734 2800 50  0000 C CNN
-F 2 "Resistor_THT:R_Axial_DIN0204_L3.6mm_D1.6mm_P5.08mm_Horizontal" V 5780 2800 50  0001 C CNN
-F 3 "~" H 5850 2800 50  0001 C CNN
-	1    5850 2800
+P 5950 2800
+F 0 "R4" V 5743 2800 50  0000 C CNN
+F 1 "100k" V 5834 2800 50  0000 C CNN
+F 2 "Resistor_SMD:R_0805_2012Metric" V 5880 2800 50  0001 C CNN
+F 3 "~" H 5950 2800 50  0001 C CNN
+	1    5950 2800
 	0    1    1    0
 $EndComp
@@
 F 0 "R1" H 3970 2746 50  0000 L CNN
 F 1 "120k" H 3970 2655 50  0000 L CNN
-F 2 "Resistor_THT:R_Axial_DIN0204_L3.6mm_D1.6mm_P5.08mm_Horizontal" V 3830 2700 50  0001 C CNN
+F 2 "Resistor_SMD:R_0805_2012Metric" V 3830 2700 50  0001 C CNN
 F 3 "~" H 3900 2700 50  0001 C CNN
 	1    3900 2700
@@
 F 0 "R2" H 3970 3396 50  0000 L CNN
 F 1 "100k" H 3970 3305 50  0000 L CNN
-F 2 "Resistor_THT:R_Axial_DIN0204_L3.6mm_D1.6mm_P5.08mm_Horizontal" V 3830 3350 50  0001 C CNN
+F 2 "Resistor_SMD:R_0805_2012Metric" V 3830 3350 50  0001 C CNN
 F 3 "~" H 3900 3350 50  0001 C CNN
 	1    3900 3350
@@
 F 0 "R3" H 4370 3396 50  0000 L CNN
 F 1 "100k" H 4370 3305 50  0000 L CNN
-F 2 "Resistor_THT:R_Axial_DIN0204_L3.6mm_D1.6mm_P5.08mm_Horizontal" V 4230 3350 50  0001 C CNN
+F 2 "Resistor_SMD:R_0805_2012Metric" V 4230 3350 50  0001 C CNN
 F 3 "~" H 4300 3350 50  0001 C CNN
 	1    4300 3350
@@
 	6500 3950 6500 4000
 Wire Wire Line
-	6000 2800 6100 2800
-Wire Wire Line
-	6000 3750 6100 3750
-Wire Wire Line
 	5300 2800 5700 2800
 Wire Wire Line
-	5200 3750 5700 3750
-Wire Wire Line
 	6500 2600 6500 2550
 Wire Wire Line
@@
 	4300 3150 5100 3150
 Wire Wire Line
-	5100 3150 5100 2150
+	5100 3150 5100 3000
 Wire Wire Line
 	5100 2150 5400 2150
@@
 Wire Wire Line
 	4300 3150 4300 3200
-Wire Wire Line
-	5400 2150 6100 2150
-Wire Wire Line
-	6100 2150 6100 2250
-Connection ~ 5400 2150
-Wire Wire Line
-	5100 3150 6100 3150
-Wire Wire Line
-	6100 3150 6100 3200
-Connection ~ 5100 3150
-Wire Wire Line
-	6100 2650 6100 2800
-Connection ~ 6100 2800
-Wire Wire Line
-	6100 2800 6200 2800
-Wire Wire Line
-	6100 3600 6100 3750
-Connection ~ 6100 3750
-Wire Wire Line
-	6100 3750 6200 3750
 Text Notes 4900 1500 0    50   ~ 0
 Connections as seen\nfrom LCD Side
@@
 F 0 "C1" H 5641 2046 50  0000 L CNN
 F 1 "10u" H 5641 1955 50  0000 L CNN
-F 2 "Capacitor_THT:C_Disc_D3.0mm_W1.6mm_P2.50mm" H 5550 2000 50  0001 C CNN
+F 2 "Capacitor_SMD:C_0805_2012Metric" H 5550 2000 50  0001 C CNN
 F 3 "~" H 5550 2000 50  0001 C CNN
 	1    5550 2000
@@
 	5100 2100 5550 2100
 Connection ~ 5100 2050
-$Comp
-L Connector_Generic:Conn_01x05 J1
-U 1 1 5B36CCA6
-P 4700 4550
-F 0 "J1" V 4573 4262 50  0000 R CNN
-F 1 "Conn_01x05" V 4664 4262 50  0000 R CNN
-F 2 "Connector_PinHeader_2.54mm:PinHeader_1x05_P2.54mm_Horizontal" H 4700 4550 50  0001 C CNN
-F 3 "~" H 4700 4550 50  0001 C CNN
-	1    4700 4550
-	0    -1   1    0
-$EndComp
 Wire Wire Line
 	3900 2500 3500 2500
-Wire Wire Line
-	3500 2500 3500 4300
-Wire Wire Line
-	3500 4300 4500 4300
-Wire Wire Line
-	4500 4300 4500 4350
 Connection ~ 3900 2500
 Wire Wire Line
@@
 	5450 3400 5450 4150
 Wire Wire Line
-	5450 3400 5800 3400
-Wire Wire Line
 	5300 2000 5300 2800
-Wire Wire Line
-	5800 2450 5350 2450
-Wire Wire Line
-	5350 2450 5350 4050
-Wire Wire Line
-	4600 4050 5350 4050
 Wire Wire Line
 	6500 2550 7300 2550
@@
 F 0 "Q1" H 4391 2946 50  0000 L CNN
 F 1 "2N3904" H 4391 2855 50  0000 L CNN
-F 2 "Package_TO_SOT_THT:TO-92_Inline" H 4400 2825 50  0001 L CIN
+F 2 "Package_TO_SOT_SMD:SOT-23" H 4400 2825 50  0001 L CIN
 F 3 "https://www.fairchildsemi.com/datasheets/2N/2N3904.pdf" H 4200 2900 50  0001 L CNN
 	1    4200 2900
@@
 F 0 "Q4" H 6591 2846 50  0000 L CNN
 F 1 "2N3904" H 6591 2755 50  0000 L CNN
-F 2 "Package_TO_SOT_THT:TO-92_Inline" H 6600 2725 50  0001 L CIN
+F 2 "Package_TO_SOT_SMD:SOT-23" H 6600 2725 50  0001 L CIN
 F 3 "https://www.fairchildsemi.com/datasheets/2N/2N3904.pdf" H 6400 2800 50  0001 L CNN
 	1    6400 2800
@@
 F 0 "Q5" H 6591 3796 50  0000 L CNN
 F 1 "2N3904" H 6591 3705 50  0000 L CNN
-F 2 "Package_TO_SOT_THT:TO-92_Inline" H 6600 3675 50  0001 L CIN
+F 2 "Package_TO_SOT_SMD:SOT-23" H 6600 3675 50  0001 L CIN
 F 3 "https://www.fairchildsemi.com/datasheets/2N/2N3904.pdf" H 6400 3750 50  0001 L CNN
 	1    6400 3750
@@
 Wire Wire Line
 	4900 4250 4900 4350
+Wire Wire Line
+	5400 2150 5700 2150
+Wire Wire Line
+	5700 2150 5700 2250
+Connection ~ 5400 2150
+Wire Wire Line
+	5700 2650 5700 2800
+Wire Wire Line
+	5700 2800 5800 2800
+Connection ~ 5700 2800
+Wire Wire Line
+	6100 2800 6200 2800
+Wire Wire Line
+	5400 2450 5400 4050
+Wire Wire Line
+	4600 4050 5400 4050
+Wire Wire Line
+	5200 3750 5750 3750
+Wire Wire Line
+	5750 3600 5750 3750
+Connection ~ 5750 3750
+Wire Wire Line
+	5750 3750 5800 3750
+Wire Wire Line
+	5100 3000 5750 3000
+Wire Wire Line
+	5750 3000 5750 3200
+Connection ~ 5100 3000
+Wire Wire Line
+	5100 3000 5100 2150
+Wire Wire Line
+	6100 3750 6200 3750
+$Comp
+L Connector_Generic:Conn_01x06 J1
+U 1 1 5B909F67
+P 4600 4550
+F 0 "J1" V 4473 4162 50  0000 R CNN
+F 1 "Conn_01x06" V 4564 4162 50  0000 R CNN
+F 2 "Connector_PinHeader_2.54mm:PinHeader_1x06_P2.54mm_Horizontal" H 4600 4550 50  0001 C CNN
+F 3 "~" H 4600 4550 50  0001 C CNN
+	1    4600 4550
+	0    -1   1    0
+$EndComp
+Wire Wire Line
+	3500 2500 3500 4150
+$Comp
+L power:GNDREF #PWR01
+U 1 1 5B90B1B9
+P 4100 4500
+F 0 "#PWR01" H 4100 4250 50  0001 C CNN
+F 1 "GNDREF" H 3900 4450 50  0000 C CNN
+F 2 "" H 4100 4500 50  0001 C CNN
+F 3 "" H 4100 4500 50  0001 C CNN
+	1    4100 4500
+	1    0    0    -1
+$EndComp
+Wire Wire Line
+	3500 4150 4400 4150
+Wire Wire Line
+	4400 4150 4400 4350
+Wire Wire Line
+	4100 4250 4500 4250
+Wire Wire Line
+	4500 4250 4500 4350
+Wire Wire Line
+	4100 4250 4100 4500
 $EndSCHEMATC

Commit message: Added Fourt Axis
Parts:
- C1: footprint Capacitor_SMD:C_0805_2012Metric -> Capacitor_SMD:C_1206_3216Metric
- R1, R2, R3, R4, R5: footprint Resistor_SMD:R_0805_2012Metric -> Resistor_SMD:R_1206_3216Metric
Changed lines of the file:
@@
 F 0 "R5" V 5743 3750 50  0000 C CNN
 F 1 "100k" V 5834 3750 50  0000 C CNN
-F 2 "Resistor_SMD:R_0805_2012Metric" V 5880 3750 50  0001 C CNN
+F 2 "Resistor_SMD:R_1206_3216Metric" V 5880 3750 50  0001 C CNN
 F 3 "~" H 5950 3750 50  0001 C CNN
 	1    5950 3750
@@
 F 0 "R4" V 5743 2800 50  0000 C CNN
 F 1 "100k" V 5834 2800 50  0000 C CNN
-F 2 "Resistor_SMD:R_0805_2012Metric" V 5880 2800 50  0001 C CNN
+F 2 "Resistor_SMD:R_1206_3216Metric" V 5880 2800 50  0001 C CNN
 F 3 "~" H 5950 2800 50  0001 C CNN
 	1    5950 2800
@@
 F 0 "R1" H 3970 2746 50  0000 L CNN
 F 1 "120k" H 3970 2655 50  0000 L CNN
-F 2 "Resistor_SMD:R_0805_2012Metric" V 3830 2700 50  0001 C CNN
+F 2 "Resistor_SMD:R_1206_3216Metric" V 3830 2700 50  0001 C CNN
 F 3 "~" H 3900 2700 50  0001 C CNN
 	1    3900 2700
@@
 F 0 "R2" H 3970 3396 50  0000 L CNN
 F 1 "100k" H 3970 3305 50  0000 L CNN
-F 2 "Resistor_SMD:R_0805_2012Metric" V 3830 3350 50  0001 C CNN
+F 2 "Resistor_SMD:R_1206_3216Metric" V 3830 3350 50  0001 C CNN
 F 3 "~" H 3900 3350 50  0001 C CNN
 	1    3900 3350
@@
 F 0 "R3" H 4370 3396 50  0000 L CNN
 F 1 "100k" H 4370 3305 50  0000 L CNN
-F 2 "Resistor_SMD:R_0805_2012Metric" V 4230 3350 50  0001 C CNN
+F 2 "Resistor_SMD:R_1206_3216Metric" V 4230 3350 50  0001 C CNN
 F 3 "~" H 4300 3350 50  0001 C CNN
 	1    4300 3350
@@
 F 0 "C1" H 5641 2046 50  0000 L CNN
 F 1 "10u" H 5641 1955 50  0000 L CNN
-F 2 "Capacitor_SMD:C_0805_2012Metric" H 5550 2000 50  0001 C CNN
+F 2 "Capacitor_SMD:C_1206_3216Metric" H 5550 2000 50  0001 C CNN
 F 3 "~" H 5550 2000 50  0001 C CNN
 	1    5550 2000
